File: Kicad/AODox.kicad_pcb (KiCad board)
At the start: 2 copper layers, 167 parts, among them J1 MCU Prog, J2 USB C Port, K0:0 KEYSW, K0:1 KEYSW, K0:10 KEYSW, K0:11 KEYSW, K0:12 KEYSW, K0:13 KEYSW, K0:14 KEYSW, K0:15 KEYSW, K0:16 KEYSW, K0:2 KEYSW, K0:3 KEYSW, K0:4 KEYSW, K0:5 KEYSW, K0:6 KEYSW, K1:0 KEYSW, K1:1 KEYSW, K1:10 KEYSW, K1:11 KEYSW, K1:12 KEYSW, K1:13 KEYSW, K1:14 KEYSW, K1:15 KEYSW, K1:16 KEYSW, K1:2 KEYSW, K1:3 KEYSW, K1:4 KEYSW, K1:5 KEYSW, K1:6 KEYSW, K1:8 KEYSW, K2:0 KEYSW, K2:1 KEYSW, K2:10 KEYSW, K2:11 KEYSW, K2:12 KEYSW, K2:13 KEYSW, K2:14 KEYSW, K2:15 KEYSW, K2:16 KEYSW, K2:2 KEYSW, K2:3 KEYSW, K2:4 KEYSW, K2:5 KEYSW, K2:6 KEYSW, K2:8 KEYSW, K3:0 KEYSW, K3:1 KEYSW, K3:11 KEYSW, K3:12 KEYSW, K3:13 KEYSW, K3:14 KEYSW, K3:15 KEYSW, K3:16 KEYSW, K3:2 KEYSW, K3:3 KEYSW, K3:4 KEYSW, K3:5 KEYSW, K3:7 KEYSW, K3:9 KEYSW, K4:0 KEYSW, K4:1 KEYSW, K4:10 KEYSW, K4:11 KEYSW, K4:12 KEYSW, K4:13 KEYSW, K4:14 KEYSW, K4:15 KEYSW, K4:16 KEYSW, K4:2 KEYSW, K4:3 KEYSW, K4:4 KEYSW, K4:5 KEYSW, K4:6 KEYSW, K4:7 KEYSW, K4:9 KEYSW, SW1 SW_Push, U1 ATMEGA32U4, X1 XTAL_18p

Commit message: [PCB] Route out traces on board
Parts:
- removed X1: XTAL_18p, Crystal:Crystal_SMD_SeikoEpson_FA238-4Pin_3.2x2.5mm_HandSoldering
- added GRAPHIC_LOGO1: Logo, PCB_logos:AODox_PCB_logo_Anurati, B.Cu at (201.2, 89.7)
- added GRAPHIC_LOGO2: PCB Edge Cuts, AODox:PCB_edgecuts, F.Cu at (165.1, 145.3)
- added Y1: XTAL_18p, Crystal:Crystal_SMD_SeikoEpson_FA238-4Pin_3.2x2.5mm_HandSoldering, F.Cu at (153.2, 100.2)
- C1, C2, C3, C4, C8, R1: moved to B.Cu
- U1: footprint Package_QFP:TQFP-44_10x10mm_P0.8mm -> keyboard_parts_AO:TQFP-44_10x10mm_P0.8mm_HandSolder
- moved J1 132.4 mm to (138.5, 80.9)
- moved C4 42.3 mm to (163.4, 104.0), turned to 0 degrees
- moved R5 38.3 mm to (156.6, 85.2)
- moved C1 37.6 mm to (168.2, 100.8), turned to 270 degrees
- moved C6 34.5 mm to (151.0, 97.5), turned to 225 degrees
- moved C7 34.2 mm to (150.5, 102.9), turned to 135 degrees
- moved R1 34.0 mm to (162.9, 97.7), turned to 180 degrees
- moved R3 32.8 mm to (166.1, 85.2)
- moved K2:16 32.1 mm to (307.6, 125.4)
- moved K1:0 32.1 mm to (28.2, 107.2)
- moved D0:16 32.1 mm to (292.1, 95.7)
- moved K3:7 32.1 mm to (148.9, 191.2)
- moved D1:0 32.1 mm to (20.9, 110.3)
- moved K1:2 32.1 mm to (71.0, 113.3)
- moved K3:2 32.1 mm to (59.8, 149.6)
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Connections:
- J1 pad 1: Net-(J1-Pad1) -> GND
- J1 pad 5: VCC -> Net-(J1-Pad5)
- J1 pad 6: GND -> VCC
- R1 pad 2: Net-(J1-Pad1) -> Net-(J1-Pad5)
- R2 pad 1: Net-(J2-PadA6) -> Net-(J2-PadA7)
- R3 pad 1: Net-(J2-PadA7) -> Net-(J2-PadA6)
- SW1 pad 2: Net-(J1-Pad1) -> Net-(J1-Pad5)
- U1 pad 13: Net-(J1-Pad1) -> Net-(J1-Pad5)
- U1 pad 18: col4 -> Net-(U1-Pad18)
- U1 pad 19: col5 -> col4
- U1 pad 20: col6 -> col5
- U1 pad 21: col7 -> col6
- U1 pad 22: row0 -> col7
- U1 pad 25: row1 -> row0
- U1 pad 26: row2 -> row1
- U1 pad 27: Net-(U1-Pad27) -> col8
- U1 pad 28: col8 -> row2
- U1 pad 3: Net-(R3-Pad2) -> Net-(R2-Pad2)
- U1 pad 4: Net-(R2-Pad2) -> Net-(R3-Pad2)
- U1 pad 7: Net-(U1-Pad7) -> VCC
Routing:
- net row4: track 0.00 -> 463.0 mm, vias 0 -> 24
- net row3: track 0.00 -> 435.3 mm, vias 0 -> 20
- net row2: track 0.00 -> 410.1 mm, vias 0 -> 19
- net row1: track 0.00 -> 368.1 mm, vias 0 -> 17
- net row0: track 0.00 -> 308.6 mm, vias 0 -> 14
- net col16: track 0.00 -> 220.4 mm, vias 0 -> 1
- net col0: track 0.00 -> 208.0 mm, vias 0 -> 1
- net col15: track 0.00 -> 193.5 mm, vias 0 -> 1
- net col1: track 0.00 -> 192.8 mm, vias 0 -> 3
- net col14: track 0.00 -> 172.6 mm, vias 0 -> 1
- net col2: track 0.00 -> 171.4 mm, vias 0 -> 3
- net col13: track 0.00 -> 152.8 mm, vias 0 -> 1
- net col3: track 0.00 -> 151.1 mm, vias 0 -> 3
- net col12: track 0.00 -> 136.8 mm, vias 0 -> 1
- net col4: track 0.00 -> 122.5 mm, vias 0 -> 1
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- added copper zone on B.Cu, net GND
- added copper zone on F.Cu, net VCC
Other:
- board outline added: 328.5 x 147.3 mm
- net class Default: clearance 0.1524 -> 0.127
- net class PWR: clearance 0.254 -> 0.127
- rule trace_clearance: 0.1524 -> 0.127

Commit message: Start versioning here at v0.2
Parts:
- moved C8 56.3 mm to (222.1, 88.6)
- moved R6 55.8 mm to (228.5, 75.3)
- moved R2 55.8 mm to (223.0, 75.3)
- moved R3 55.8 mm to (221.0, 75.3)
- moved R5 55.8 mm to (211.5, 75.3)
- moved R1 55.7 mm to (217.8, 88.6)
- moved K2:15 55.6 mm to (339.9, 123.2)
- moved K3:2 55.6 mm to (114.7, 140.5)
- moved K1:11 55.6 mm to (260.1, 122.0)
- moved U1 55.6 mm to (220.0, 91.8)
- moved K0:15 55.6 mm to (328.8, 86.8)
- moved K3:5 55.6 mm to (168.9, 158.4)
- moved K3:12 55.6 mm to (289.0, 151.6)
- moved D0:11 55.6 mm to (250.1, 110.5)
- moved D0:6 55.6 mm to (196.3, 112.5)
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Connections:
- U1 pad 29: Net-(U1-Pad29) -> row3
- U1 pad 30: row3 -> row4
- U1 pad 31: row4 -> col9
- U1 pad 32: col9 -> Net-(U1-Pad32)
Routing:
- net col6: track 101.6 -> 97.9 mm
- net row3: track 435.3 -> 438.3 mm
- net row4: track 463.0 -> 462.1 mm
- net Net-(J2-PadB5): track 15.3 -> 14.5 mm
- net Net-(R2-Pad2): track 8.82 -> 9.52 mm
- net Net-(J2-PadA6): track 9.54 -> 8.84 mm
- net Net-(R3-Pad2): track 8.82 -> 9.52 mm
- net Net-(J2-PadA7): track 9.54 -> 8.84 mm
- net col3: track 151.1 -> 150.4 mm
- net col1: track 192.8 -> 192.3 mm
- net row2: track 410.1 -> 410.6 mm
- net col2: track 171.4 -> 170.9 mm
