File: Kicad/AODox.sch (KiCad schematic (older format))
At the start: 19 parts

Commit message: Update schematic annotations
Parts:
- gave numbers to parts that had none: 19
Connections:
- net labels added: col0, col1, col10, col11, col12, col13, col14, col15, col16, col2, col3, col4, col5, col6, col7, col8, col9, row0, row1, row2, row3, row4
- wire segments 72 -> 75
- no-connect marks 3 -> 7
Changed lines of the file:
@@
 $EndDescr
 $Comp
-L AODox:ATMEGA32U4 U?
+L AODox:ATMEGA32U4 U1
 U 1 1 5DAE27ED
 P 6000 3900
-F 0 "U?" V 5900 3875 60  0000 L CNN
+F 0 "U1" V 5900 3875 60  0000 L CNN
 F 1 "ATMEGA32U4" V 6025 3625 60  0000 L CNN
 F 2 "" H 6000 3900 60  0000 C CNN
@@
 $EndComp
 $Comp
-L Connector:USB_C_Receptacle_USB2.0 J?
+L Connector:USB_C_Receptacle_USB2.0 J2
 U 1 1 5DAE85C1
 P 6300 950
-F 0 "J?" V 6225 1700 50  0000 L CNN
+F 0 "J2" V 6225 1700 50  0000 L CNN
 F 1 "USB C Port" V 6350 1700 50  0000 L CNN
 F 2 "" H 6450 950 50  0001 C CNN
@@
 $EndComp
 $Comp
-L keyboard_parts:XTAL_GND X?
+L keyboard_parts:XTAL_GND X1
 U 1 1 5DAEEB3A
 P 3850 3900
-F 0 "X?" H 3950 3750 60  0000 C CNN
+F 0 "X1" H 3950 3750 60  0000 C CNN
 F 1 "XTAL_18p" H 3875 4050 60  0000 C CNN
 F 2 "" H 3850 3900 60  0000 C CNN
@@
 $EndComp
 $Comp
-L Device:C_Small C?
+L Device:C_Small C7
 U 1 1 5DAEF537
 P 4200 4100
-F 0 "C?" H 4225 4175 50  0000 L CNN
+F 0 "C7" H 4225 4175 50  0000 L CNN
 F 1 "22p" H 4225 4025 50  0000 L CNN
 F 2 "" H 4200 4100 50  0001 C CNN
@@
 $EndComp
 $Comp
-L Device:C_Small C?
+L Device:C_Small C6
 U 1 1 5DAF087A
 P 3500 4100
-F 0 "C?" H 3525 4175 50  0000 L CNN
+F 0 "C6" H 3525 4175 50  0000 L CNN
 F 1 "22p" H 3525 4025 50  0000 L CNN
 F 2 "" H 3500 4100 50  0001 C CNN
@@
 $EndComp
 $Comp
-L power:GND #PWR?
+L power:GND #PWR04
 U 1 1 5DAF2AC6
 P 3850 4350
-F 0 "#PWR?" H 3850 4100 50  0001 C CNN
+F 0 "#PWR04" H 3850 4100 50  0001 C CNN
 F 1 "GND" H 3855 4177 50  0000 C CNN
 F 2 "" H 3850 4350 50  0001 C CNN
@@
 $EndComp
 $Comp
-L Device:C_Small C?
+L Device:C_Small C1
 U 1 1 5DAF6260
 P 2350 2650
-F 0 "C?" H 2375 2725 50  0000 L CNN
+F 0 "C1" H 2375 2725 50  0000 L CNN
 F 1 "0.1u" H 2375 2575 50  0000 L CNN
 F 2 "" H 2350 2650 50  0001 C CNN
@@
 $EndComp
 $Comp
-L Device:C_Small C?
+L Device:C_Small C2
 U 1 1 5DAF8777
 P 2600 2650
-F 0 "C?" H 2625 2725 50  0000 L CNN
+F 0 "C2" H 2625 2725 50  0000 L CNN
 F 1 "0.1u" H 2625 2575 50  0000 L CNN
 F 2 "" H 2600 2650 50  0001 C CNN
@@
 $EndComp
 $Comp
-L Device:C_Small C?
+L Device:C_Small C3
 U 1 1 5DAF8AF0
 P 2850 2650
-F 0 "C?" H 2875 2725 50  0000 L CNN
+F 0 "C3" H 2875 2725 50  0000 L CNN
 F 1 "0.1u" H 2875 2575 50  0000 L CNN
 F 2 "" H 2850 2650 50  0001 C CNN
@@
 $EndComp
 $Comp
-L Device:C_Small C?
+L Device:C_Small C4
 U 1 1 5DAF8E8B
 P 3100 2650
-F 0 "C?" H 3125 2725 50  0000 L CNN
+F 0 "C4" H 3125 2725 50  0000 L CNN
 F 1 "0.1u" H 3125 2575 50  0000 L CNN
 F 2 "" H 3100 2650 50  0001 C CNN
@@
 $EndComp
 $Comp
-L Device:C_Small C?
+L Device:C_Small C5
 U 1 1 5DAF9226
 P 3350 2650
-F 0 "C?" H 3375 2725 50  0000 L CNN
+F 0 "C5" H 3375 2725 50  0000 L CNN
 F 1 "4.7u" H 3375 2575 50  0000 L CNN
 F 2 "" H 3350 2650 50  0001 C CNN
@@
 $EndComp
 $Comp
-L power:GND #PWR?
+L power:GND #PWR02
 U 1 1 5DAF971E
 P 2350 2950
-F 0 "#PWR?" H 2350 2700 50  0001 C CNN
+F 0 "#PWR02" H 2350 2700 50  0001 C CNN
 F 1 "GND" H 2355 2777 50  0000 C CNN
 F 2 "" H 2350 2950 50  0001 C CNN
@@
 	2350 2550 2350 2450
 $Comp
-L power:VCC #PWR?
+L power:VCC #PWR01
 U 1 1 5DAFA77E
 P 2350 2350
-F 0 "#PWR?" H 2350 2200 50  0001 C CNN
+F 0 "#PWR01" H 2350 2200 50  0001 C CNN
 F 1 "VCC" H 2367 2523 50  0000 C CNN
 F 2 "" H 2350 2350 50  0001 C CNN
@@
 	3550 3500 3650 3500
 $Comp
-L power:VCC #PWR?
+L power:VCC #PWR05
 U 1 1 5DB0B43C
 P 4150 3100
-F 0 "#PWR?" H 4150 2950 50  0001 C CNN
+F 0 "#PWR05" H 4150 2950 50  0001 C CNN
 F 1 "VCC" H 4167 3273 50  0000 C CNN
 F 2 "" H 4150 3100 50  0001 C CNN
@@
 $EndComp
 $Comp
-L power:GND #PWR?
+L power:GND #PWR03
 U 1 1 5DB0AD48
 P 3550 3500
-F 0 "#PWR?" H 3550 3250 50  0001 C CNN
+F 0 "#PWR03" H 3550 3250 50  0001 C CNN
 F 1 "GND" V 3555 3372 50  0000 R CNN
 F 2 "" H 3550 3500 50  0001 C CNN
@@
 $EndComp
 $Comp
-L Switch:SW_Push SW?
+L Switch:SW_Push SW1
 U 1 1 5DB09B68
 P 3850 3500
-F 0 "SW?" H 3850 3650 50  0000 C CNN
+F 0 "SW1" H 3850 3650 50  0000 C CNN
 F 1 "SW_Push" H 3850 3450 50  0000 C CNN
 F 2 "" H 3850 3700 50  0001 C CNN
@@
 Connection ~ 4150 3500
 $Comp
-L Device:R_Small R?
+L Device:R_Small R1
 U 1 1 5DB0A7CA
 P 4150 3300
-F 0 "R?" H 4209 3346 50  0000 L CNN
+F 0 "R1" H 4209 3346 50  0000 L CNN
 F 1 "10k" H 4209 3255 50  0000 L CNN
 F 2 "" H 4150 3300 50  0001 C CNN
@@
 $EndComp
 $Comp
-L Device:R_Small R?
+L Device:R_Small R4
 U 1 1 5DB181EB
 P 6500 5400
-F 0 "R?" H 6559 5446 50  0000 L CNN
+F 0 "R4" H 6559 5446 50  0000 L CNN
 F 1 "10k" H 6559 5355 50  0000 L CNN
 F 2 "" H 6500 5400 50  0001 C CNN
@@
 $EndComp
 $Comp
-L power:GND #PWR?
+L power:GND #PWR08
 U 1 1 5DB19020
 P 6500 5600
-F 0 "#PWR?" H 6500 5350 50  0001 C CNN
+F 0 "#PWR08" H 6500 5350 50  0001 C CNN
 F 1 "GND" H 6505 5427 50  0000 C CNN
 F 2 "" H 6500 5600 50  0001 C CNN
@@
 	6300 1550 6400 1550
 $Comp
-L power:GND #PWR?
+L power:GND #PWR06
 U 1 1 5DB1C0A7
 P 5300 950
-F 0 "#PWR?" H 5300 700 50  0001 C CNN
+F 0 "#PWR06" H 5300 700 50  0001 C CNN
 F 1 "GND" H 5305 777 50  0000 C CNN
 F 2 "" H 5300 950 50  0001 C CNN
@@
 NoConn ~ 5800 1550
 $Comp
-L Device:R R?
+L Device:R R5
 U 1 1 5DB2D6C5
 P 6600 1800
-F 0 "R?" H 6450 1800 50  0000 L CNN
+F 0 "R5" H 6450 1800 50  0000 L CNN
 F 1 "5.1k" V 6600 1700 50  0000 L CNN
 F 2 "" V 6530 1800 50  0001 C CNN
@@
 $EndComp
 $Comp
-L Device:R R?
+L Device:R R6
 U 1 1 5DB2E11A
 P 6700 1800
-F 0 "R?" H 6750 1800 50  0000 L CNN
+F 0 "R6" H 6750 1800 50  0000 L CNN
 F 1 "5.1k" V 6700 1700 50  0000 L CNN
 F 2 "" V 6630 1800 50  0001 C CNN
@@
 $EndComp
 $Comp
-L power:GND #PWR?
+L power:GND #PWR09
 U 1 1 5DB2E530
 P 6650 2050
-F 0 "#PWR?" H 6650 1800 50  0001 C CNN
+F 0 "#PWR09" H 6650 1800 50  0001 C CNN
 F 1 "GND" H 6655 1877 50  0000 C CNN
 F 2 "" H 6650 2050 50  0001 C CNN
@@
 	6700 1650 6700 1550
 $Comp
-L Device:R R?
+L Device:R R2
 U 1 1 5DB31C0A
 P 6200 2050
-F 0 "R?" H 6050 2050 50  0000 L CNN
+F 0 "R2" H 6050 2050 50  0000 L CNN
 F 1 "22" V 6200 2000 50  0000 L CNN
 F 2 "" V 6130 2050 50  0001 C CNN
@@
 $EndComp
 $Comp
-L Device:R R?
+L Device:R R3
 U 1 1 5DB32FF9
 P 6300 2050
-F 0 "R?" H 6350 2050 50  0000 L CNN
+F 0 "R3" H 6350 2050 50  0000 L CNN
 F 1 "22" V 6300 2000 50  0000 L CNN
 F 2 "" V 6230 2050 50  0001 C CNN
@@
 	6200 2200 6200 2600
 $Comp
-L power:VCC #PWR?
+L power:VCC #PWR010
 U 1 1 5DB3945C
 P 7200 1550
-F 0 "#PWR?" H 7200 1400 50  0001 C CNN
+F 0 "#PWR010" H 7200 1400 50  0001 C CNN
 F 1 "VCC" H 7217 1723 50  0000 C CNN
 F 2 "" H 7200 1550 50  0001 C CNN
@@
 Connection ~ 6900 1550
 $Comp
-L Device:C_Small C?
+L Device:C_Small C8
 U 1 1 5DB3C818
 P 6000 2400
-F 0 "C?" H 5900 2475 50  0000 L CNN
+F 0 "C8" H 5900 2475 50  0000 L CNN
 F 1 "1u" H 5875 2325 50  0000 L CNN
 F 2 "" H 6000 2400 50  0001 C CNN
@@
 $EndComp
 $Comp
-L power:GND #PWR?
+L power:GND #PWR07
 U 1 1 5DB3D6B5
 P 6000 2200
-F 0 "#PWR?" H 6000 1950 50  0001 C CNN
+F 0 "#PWR07" H 6000 1950 50  0001 C CNN
 F 1 "GND" V 6005 2072 50  0000 R CNN
 F 2 "" H 6000 2200 50  0001 C CNN
@@
 	4150 3500 4450 3500
 $Comp
-L Connector:Conn_01x06_Male J?
+L Connector:Conn_01x06_Male J1
 U 1 1 5DB41B5C
 P 4650 1800
-F 0 "J?" V 4725 1425 50  0000 R CNN
+F 0 "J1" V 4725 1425 50  0000 R CNN
 F 1 "MCU Prog" V 4575 1950 50  0000 R CNN
 F 2 "" H 4650 1800 50  0001 C CNN
@@
 F1 "key_matrix.sch" 50
 $EndSheet
+NoConn ~ 7300 3600
+Text GLabel 6500 2600 2    50   BiDi ~ 0
+col16
+Text GLabel 7300 3700 2    50   BiDi ~ 0
+col15
+Text GLabel 7300 3800 2    50   BiDi ~ 0
+col14
+Text GLabel 7300 3900 2    50   BiDi ~ 0
+col13
+Text GLabel 7300 4000 2    50   BiDi ~ 0
+col12
+Text GLabel 7300 4100 2    50   BiDi ~ 0
+col11
+Text GLabel 7300 4200 2    50   BiDi ~ 0
+col10
+Text GLabel 6400 5200 3    50   BiDi ~ 0
+col9
+Text GLabel 5800 2600 1    50   BiDi ~ 0
+col0
+Wire Wire Line
+	5700 2400 5700 2150
+Connection ~ 5700 2400
+Wire Wire Line
+	5600 2500 5600 2150
+Connection ~ 5600 2500
+Wire Wire Line
+	5500 2600 5500 2150
+Connection ~ 5500 2600
+Text GLabel 5700 2150 1    50   BiDi ~ 0
+col1
+Text GLabel 5600 2150 1    50   BiDi ~ 0
+col2
+Text GLabel 5500 2150 1    50   BiDi ~ 0
+col3
+NoConn ~ 4700 3400
+Text GLabel 4700 4000 0    50   BiDi ~ 0
+col4
+Text GLabel 4700 4100 0    50   BiDi ~ 0
+col5
+Text GLabel 4700 4200 0    50   BiDi ~ 0
+col6
+Text GLabel 4700 4300 0    50   BiDi ~ 0
+col7
+Text GLabel 4700 4400 0    50   BiDi ~ 0
+row0
+Text GLabel 5700 5200 3    50   BiDi ~ 0
+row1
+Text GLabel 5800 5200 3    50   BiDi ~ 0
+row2
+Text GLabel 6000 5200 3    50   BiDi ~ 0
+col8
+Text GLabel 6200 5200 3    50   BiDi ~ 0
+row3
+Text GLabel 6300 5200 3    50   BiDi ~ 0
+row4
+NoConn ~ 5900 5200
+NoConn ~ 6100 5200
 $EndSCHEMATC

Commit message: Assign footprints to schematic symbols
Parts:
- C1, C2, C3, C4, C5, C6, C7, C8: footprint (none) -> Capacitor_SMD:C_0805_2012Metric_Pad1.15x1.40mm_HandSolder
- J1: footprint (none) -> Connector_PinHeader_2.54mm:PinHeader_1x06_P2.54mm_Vertical
- J2: footprint (none) -> Connector_USB:USB_C_Receptacle_GCT_USB4085
- R1, R2, R3, R4, R5, R6: footprint (none) -> Resistor_SMD:R_0805_2012Metric_Pad1.15x1.40mm_HandSolder
Changed lines of the file:
@@
 F 0 "U1" V 5900 3875 60  0000 L CNN
 F 1 "ATMEGA32U4" V 6025 3625 60  0000 L CNN
-F 2 "" H 6000 3900 60  0000 C CNN
+F 2 "" H 6000 3900 60  0001 C CNN
 F 3 "" H 6000 3900 60  0000 C CNN
 	1    6000 3900
@@
 F 0 "J2" V 6225 1700 50  0000 L CNN
 F 1 "USB C Port" V 6350 1700 50  0000 L CNN
-F 2 "" H 6450 950 50  0001 C CNN
+F 2 "Connector_USB:USB_C_Receptacle_GCT_USB4085" H 6450 950 50  0001 C CNN
 F 3 "https://www.usb.org/sites/default/files/documents/usb_type-c.zip" H 6450 950 50  0001 C CNN
 	1    6300 950
@@
 F 0 "X1" H 3950 3750 60  0000 C CNN
 F 1 "XTAL_18p" H 3875 4050 60  0000 C CNN
-F 2 "" H 3850 3900 60  0000 C CNN
+F 2 "" H 3850 3900 60  0001 C CNN
 F 3 "" H 3850 3900 60  0000 C CNN
 	1    3850 3900
@@
 F 0 "C7" H 4225 4175 50  0000 L CNN
 F 1 "22p" H 4225 4025 50  0000 L CNN
-F 2 "" H 4200 4100 50  0001 C CNN
+F 2 "Capacitor_SMD:C_0805_2012Metric_Pad1.15x1.40mm_HandSolder" H 4200 4100 50  0001 C CNN
 F 3 "~" H 4200 4100 50  0001 C CNN
 	1    4200 4100
@@
 F 0 "C6" H 3525 4175 50  0000 L CNN
 F 1 "22p" H 3525 4025 50  0000 L CNN
-F 2 "" H 3500 4100 50  0001 C CNN
+F 2 "Capacitor_SMD:C_0805_2012Metric_Pad1.15x1.40mm_HandSolder" H 3500 4100 50  0001 C CNN
 F 3 "~" H 3500 4100 50  0001 C CNN
 	1    3500 4100
@@
 F 0 "C1" H 2375 2725 50  0000 L CNN
 F 1 "0.1u" H 2375 2575 50  0000 L CNN
-F 2 "" H 2350 2650 50  0001 C CNN
+F 2 "Capacitor_SMD:C_0805_2012Metric_Pad1.15x1.40mm_HandSolder" H 2350 2650 50  0001 C CNN
 F 3 "~" H 2350 2650 50  0001 C CNN
 	1    2350 2650
@@
 F 0 "C2" H 2625 2725 50  0000 L CNN
 F 1 "0.1u" H 2625 2575 50  0000 L CNN
-F 2 "" H 2600 2650 50  0001 C CNN
+F 2 "Capacitor_SMD:C_0805_2012Metric_Pad1.15x1.40mm_HandSolder" H 2600 2650 50  0001 C CNN
 F 3 "~" H 2600 2650 50  0001 C CNN
 	1    2600 2650
@@
 F 0 "C3" H 2875 2725 50  0000 L CNN
 F 1 "0.1u" H 2875 2575 50  0000 L CNN
-F 2 "" H 2850 2650 50  0001 C CNN
+F 2 "Capacitor_SMD:C_0805_2012Metric_Pad1.15x1.40mm_HandSolder" H 2850 2650 50  0001 C CNN
 F 3 "~" H 2850 2650 50  0001 C CNN
 	1    2850 2650
@@
 F 0 "C4" H 3125 2725 50  0000 L CNN
 F 1 "0.1u" H 3125 2575 50  0000 L CNN
-F 2 "" H 3100 2650 50  0001 C CNN
+F 2 "Capacitor_SMD:C_0805_2012Metric_Pad1.15x1.40mm_HandSolder" H 3100 2650 50  0001 C CNN
 F 3 "~" H 3100 2650 50  0001 C CNN
 	1    3100 2650
@@
 F 0 "C5" H 3375 2725 50  0000 L CNN
 F 1 "4.7u" H 3375 2575 50  0000 L CNN
-F 2 "" H 3350 2650 50  0001 C CNN
+F 2 "Capacitor_SMD:C_0805_2012Metric_Pad1.15x1.40mm_HandSolder" H 3350 2650 50  0001 C CNN
 F 3 "~" H 3350 2650 50  0001 C CNN
 	1    3350 2650
@@
 F 0 "R1" H 4209 3346 50  0000 L CNN
 F 1 "10k" H 4209 3255 50  0000 L CNN
-F 2 "" H 4150 3300 50  0001 C CNN
+F 2 "Resistor_SMD:R_0805_2012Metric_Pad1.15x1.40mm_HandSolder" H 4150 3300 50  0001 C CNN
 F 3 "~" H 4150 3300 50  0001 C CNN
 	1    4150 3300
@@
 F 0 "R4" H 6559 5446 50  0000 L CNN
 F 1 "10k" H 6559 5355 50  0000 L CNN
-F 2 "" H 6500 5400 50  0001 C CNN
+F 2 "Resistor_SMD:R_0805_2012Metric_Pad1.15x1.40mm_HandSolder" H 6500 5400 50  0001 C CNN
 F 3 "~" H 6500 5400 50  0001 C CNN
 	1    6500 5400
@@
 F 0 "R5" H 6450 1800 50  0000 L CNN
 F 1 "5.1k" V 6600 1700 50  0000 L CNN
-F 2 "" V 6530 1800 50  0001 C CNN
+F 2 "Resistor_SMD:R_0805_2012Metric_Pad1.15x1.40mm_HandSolder" V 6530 1800 50  0001 C CNN
 F 3 "~" H 6600 1800 50  0001 C CNN
 	1    6600 1800
@@
 F 0 "R6" H 6750 1800 50  0000 L CNN
 F 1 "5.1k" V 6700 1700 50  0000 L CNN
-F 2 "" V 6630 1800 50  0001 C CNN
+F 2 "Resistor_SMD:R_0805_2012Metric_Pad1.15x1.40mm_HandSolder" V 6630 1800 50  0001 C CNN
 F 3 "~" H 6700 1800 50  0001 C CNN
 	1    6700 1800
@@
 F 0 "R2" H 6050 2050 50  0000 L CNN
 F 1 "22" V 6200 2000 50  0000 L CNN
-F 2 "" V 6130 2050 50  0001 C CNN
+F 2 "Resistor_SMD:R_0805_2012Metric_Pad1.15x1.40mm_HandSolder" V 6130 2050 50  0001 C CNN
 F 3 "~" H 6200 2050 50  0001 C CNN
 	1    6200 2050
@@
 F 0 "R3" H 6350 2050 50  0000 L CNN
 F 1 "22" V 6300 2000 50  0000 L CNN
-F 2 "" V 6230 2050 50  0001 C CNN
+F 2 "Resistor_SMD:R_0805_2012Metric_Pad1.15x1.40mm_HandSolder" V 6230 2050 50  0001 C CNN
 F 3 "~" H 6300 2050 50  0001 C CNN
 	1    6300 2050
@@
 F 0 "C8" H 5900 2475 50  0000 L CNN
 F 1 "1u" H 5875 2325 50  0000 L CNN
-F 2 "" H 6000 2400 50  0001 C CNN
+F 2 "Capacitor_SMD:C_0805_2012Metric_Pad1.15x1.40mm_HandSolder" H 6000 2400 50  0001 C CNN
 F 3 "~" H 6000 2400 50  0001 C CNN
 	1    6000 2400
@@
 F 0 "J1" V 4725 1425 50  0000 R CNN
 F 1 "MCU Prog" V 4575 1950 50  0000 R CNN
-F 2 "" H 4650 1800 50  0001 C CNN
+F 2 "Connector_PinHeader_2.54mm:PinHeader_1x06_P2.54mm_Vertical" H 4650 1800 50  0001 C CNN
 F 3 "~" H 4650 1800 50  0001 C CNN
 	1    4650 1800

Commit message: Rough out PCB layout
Parts:
- SW1: footprint (none) -> Button_Switch_SMD:SW_SPST_CK_KXT3
- U1: footprint (none) -> Package_QFP:TQFP-44_10x10mm_P0.8mm
- X1: footprint (none) -> Crystal:Crystal_SMD_SeikoEpson_FA238-4Pin_3.2x2.5mm_HandSoldering
Changed lines of the file:
@@
 Title "AODox"
 Date "2019-10-21"
-Rev "v1"
+Rev "v2"
 Comp "AO Industries"
 Comment1 ""
@@
 F 0 "U1" V 5900 3875 60  0000 L CNN
 F 1 "ATMEGA32U4" V 6025 3625 60  0000 L CNN
-F 2 "" H 6000 3900 60  0001 C CNN
+F 2 "Package_QFP:TQFP-44_10x10mm_P0.8mm" H 6000 3900 60  0001 C CNN
 F 3 "" H 6000 3900 60  0000 C CNN
 	1    6000 3900
@@
 F 0 "X1" H 3950 3750 60  0000 C CNN
 F 1 "XTAL_18p" H 3875 4050 60  0000 C CNN
-F 2 "" H 3850 3900 60  0001 C CNN
+F 2 "Crystal:Crystal_SMD_SeikoEpson_FA238-4Pin_3.2x2.5mm_HandSoldering" H 3850 3900 60  0001 C CNN
 F 3 "" H 3850 3900 60  0000 C CNN
 	1    3850 3900
@@
 F 0 "SW1" H 3850 3650 50  0000 C CNN
 F 1 "SW_Push" H 3850 3450 50  0000 C CNN
-F 2 "" H 3850 3700 50  0001 C CNN
+F 2 "Button_Switch_SMD:SW_SPST_CK_KXT3" H 3850 3700 50  0001 C CNN
 F 3 "~" H 3850 3700 50  0001 C CNN
 	1    3850 3500

Commit message: Start versioning here at v0.2
Parts:
- removed X1: XTAL_18p, Crystal:Crystal_SMD_SeikoEpson_FA238-4Pin_3.2x2.5mm_HandSoldering, symbol keyboard_parts:XTAL_GND
- added GRAPHIC_LOGO1: Logo, PCB_logos:AODox_PCB_logo_Anurati, symbol keyboard_parts_AO:Graphic_Logo
- added GRAPHIC_LOGO2: PCB Edge Cuts, AODox:PCB_edgecuts, symbol keyboard_parts_AO:Graphic_Logo
- added Y1: XTAL_18p, Crystal:Crystal_SMD_SeikoEpson_FA238-4Pin_3.2x2.5mm_HandSoldering, symbol Device:Crystal_GND24_Small
- U1: footprint Package_QFP:TQFP-44_10x10mm_P0.8mm -> keyboard_parts_AO:TQFP-44_10x10mm_P0.8mm_HandSolder
Connections:
- wire segments 75 -> 78
Other:
- moved on the sheet: C1, C2, C3, C4, C5, C6, C7, C8, J1, J2, R1, R2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

Commit message: Commit before pulling in from origin
Parts:
- C1, C2, C3, C4, C5, C6, C7, C8: symbol Device:C_Small -> AODox-rescue:C_Small-Device
- GRAPHIC_LOGO1, GRAPHIC_LOGO2: symbol keyboard_parts_AO:Graphic_Logo -> AODox-rescue:Graphic_Logo-keyboard_parts_AO
- J1: symbol Connector:Conn_01x06_Male -> AODox-rescue:Conn_01x06_Male-Connector
- J2: symbol Connector:USB_C_Receptacle_USB2.0 -> AODox-rescue:USB_C_Receptacle_USB2.0-Connector
- R1, R4: symbol Device:R_Small -> AODox-rescue:R_Small-Device
- R2, R3, R5, R6: symbol Device:R -> AODox-rescue:R-Device
- SW1: symbol Switch:SW_Push -> AODox-rescue:SW_Push-Switch
- Y1: symbol Device:Crystal_GND24_Small -> AODox-rescue:Crystal_GND24_Small-Device
Changed lines of the file:
@@
 EESchema Schematic File Version 4
-LIBS:AODox-cache
 EELAYER 30 0
 EELAYER END
@@
 $EndDescr
 $Comp
-L Connector:USB_C_Receptacle_USB2.0 J2
+L AODox-rescue:USB_C_Receptacle_USB2.0-Connector J2
 U 1 1 5DAE85C1
 P 6300 1600
@@
 $EndComp
 $Comp
-L Device:C_Small C7
+L AODox-rescue:C_Small-Device C7
 U 1 1 5DAEF537
 P 4200 4750
@@
 $EndComp
 $Comp
-L Device:C_Small C6
+L AODox-rescue:C_Small-Device C6
 U 1 1 5DAF087A
 P 3500 4750
@@
 $EndComp
 $Comp
-L power:GND #PWR04
+L AODox-rescue:GND-power #PWR04
 U 1 1 5DAF2AC6
 P 3850 5000
@@
 $EndComp
 $Comp
-L Device:C_Small C1
+L AODox-rescue:C_Small-Device C1
 U 1 1 5DAF6260
 P 2350 3300
@@
 $EndComp
 $Comp
-L Device:C_Small C2
+L AODox-rescue:C_Small-Device C2
 U 1 1 5DAF8777
 P 2600 3300
@@
 $EndComp
 $Comp
-L Device:C_Small C3
+L AODox-rescue:C_Small-Device C3
 U 1 1 5DAF8AF0
 P 2850 3300
@@
 $EndComp
 $Comp
-L Device:C_Small C4
+L AODox-rescue:C_Small-Device C4
 U 1 1 5DAF8E8B
 P 3100 3300
@@
 $EndComp
 $Comp
-L Device:C_Small C5
+L AODox-rescue:C_Small-Device C5
 U 1 1 5DAF9226
 P 3350 3300
@@
 $EndComp
 $Comp
-L power:GND #PWR02
+L AODox-rescue:GND-power #PWR02
 U 1 1 5DAF971E
 P 2350 3600
@@
 	2350 3200 2350 3100
 $Comp
-L power:VCC #PWR01
+L AODox-rescue:VCC-power #PWR01
 U 1 1 5DAFA77E
 P 2350 3000
@@
 	3550 4150 3650 4150
 $Comp
-L power:VCC #PWR05
+L AODox-rescue:VCC-power #PWR05
 U 1 1 5DB0B43C
 P 4150 3750
@@
 $EndComp
 $Comp
-L power:GND #PWR03
+L AODox-rescue:GND-power #PWR03
 U 1 1 5DB0AD48
 P 3550 4150
@@
 $EndComp
 $Comp
-L Switch:SW_Push SW1
+L AODox-rescue:SW_Push-Switch SW1
 U 1 1 5DB09B68
 P 3850 4150
@@
 Connection ~ 4150 4150
 $Comp
-L Device:R_Small R1
+L AODox-rescue:R_Small-Device R1
 U 1 1 5DB0A7CA
 P 4150 3950
@@
 $EndComp
 $Comp
-L Device:R_Small R4
+L AODox-rescue:R_Small-Device R4
 U 1 1 5DB181EB
 P 6500 6050
@@
 $EndComp
 $Comp
-L power:GND #PWR08
+L AODox-rescue:GND-power #PWR08
 U 1 1 5DB19020
 P 6500 6250
@@
 	6300 2200 6400 2200
 $Comp
-L power:GND #PWR06
+L AODox-rescue:GND-power #PWR06
 U 1 1 5DB1C0A7
 P 5300 1600
@@
 NoConn ~ 5800 2200
 $Comp
-L Device:R R5
+L AODox-rescue:R-Device R5
 U 1 1 5DB2D6C5
 P 6600 2450
@@
 $EndComp
 $Comp
-L Device:R R6
+L AODox-rescue:R-Device R6
 U 1 1 5DB2E11A
 P 6700 2450
@@
 $EndComp
 $Comp
-L power:GND #PWR09
+L AODox-rescue:GND-power #PWR09
 U 1 1 5DB2E530
 P 6650 2700
@@
 	6700 2300 6700 2200
 $Comp
-L Device:R R3
+L AODox-rescue:R-Device R3
 U 1 1 5DB32FF9
 P 6200 2700
@@
 	6200 2850 6200 3250
 $Comp
-L power:VCC #PWR010
+L AODox-rescue:VCC-power #PWR010
 U 1 1 5DB3945C
 P 7200 2200
@@
 Connection ~ 6900 2200
 $Comp
-L Device:C_Small C8
+L AODox-rescue:C_Small-Device C8
 U 1 1 5DB3C818
 P 6000 2650
@@
 $EndComp
 $Comp
-L power:GND #PWR07
+L AODox-rescue:GND-power #PWR07
 U 1 1 5DB3D6B5
 P 6000 2400
@@
 GND
 $Comp
-L Connector:Conn_01x06_Male J1
+L AODox-rescue:Conn_01x06_Male-Connector J1
 U 1 1 5DB41B5C
 P 4650 2450
@@
 GND
 $Comp
-L Device:Crystal_GND24_Small Y1
+L AODox-rescue:Crystal_GND24_Small-Device Y1
 U 1 1 5DB7805D
 P 3850 4550
@@
 	6000 2550 6000 2400
 $Comp
-L power:VCC #PWR0101
+L AODox-rescue:VCC-power #PWR0101
 U 1 1 5DD2E542
 P 5900 3050
@@
 	5900 3250 5900 3050
 $Comp
-L keyboard_parts_AO:Graphic_Logo GRAPHIC_LOGO1
+L AODox-rescue:Graphic_Logo-keyboard_parts_AO GRAPHIC_LOGO1
 U 1 1 5DD2CCD1
 P 9100 3400
@@
 $EndComp
 $Comp
-L keyboard_parts_AO:Graphic_Logo GRAPHIC_LOGO2
+L AODox-rescue:Graphic_Logo-keyboard_parts_AO GRAPHIC_LOGO2
 U 1 1 5DD2D5B8
 P 9100 3950
@@
 $EndComp
 $Comp
-L Device:R R2
+L AODox-rescue:R-Device R2
 U 1 1 5DB31C0A
 P 6300 2700
