File: Kicad/key_matrix.sch (KiCad schematic (older format))
At the start: 154 parts, among them K0:0 KEYSW, K0:1 KEYSW, K0:10 KEYSW, K0:11 KEYSW, K0:12 KEYSW, K0:13 KEYSW, K0:14 KEYSW, K0:15 KEYSW, K0:16 KEYSW, K0:2 KEYSW, K0:3 KEYSW, K0:4 KEYSW, K0:5 KEYSW, K0:6 KEYSW, K0:8 KEYSW, K1:0 KEYSW, K1:1 KEYSW, K1:10 KEYSW, K1:11 KEYSW, K1:12 KEYSW, K1:13 KEYSW, K1:14 KEYSW, K1:15 KEYSW, K1:16 KEYSW, K1:2 KEYSW, K1:3 KEYSW, K1:4 KEYSW, K1:5 KEYSW, K1:6 KEYSW, K1:8 KEYSW, K2:0 KEYSW, K2:1 KEYSW, K2:10 KEYSW, K2:11 KEYSW, K2:12 KEYSW, K2:13 KEYSW, K2:14 KEYSW, K2:15 KEYSW, K2:16 KEYSW, K2:2 KEYSW, K2:3 KEYSW, K2:4 KEYSW, K2:5 KEYSW, K2:6 KEYSW, K2:8 KEYSW, K3:0 KEYSW, K3:1 KEYSW, K3:11 KEYSW, K3:12 KEYSW, K3:13 KEYSW, K3:14 KEYSW, K3:15 KEYSW, K3:16 KEYSW, K3:2 KEYSW, K3:3 KEYSW, K3:4 KEYSW, K3:5 KEYSW, K3:7 KEYSW, K3:8 KEYSW, K3:9 KEYSW, K4:0 KEYSW, K4:1 KEYSW, K4:10 KEYSW, K4:11 KEYSW, K4:12 KEYSW, K4:13 KEYSW, K4:14 KEYSW, K4:15 KEYSW, K4:16 KEYSW, K4:2 KEYSW, K4:3 KEYSW, K4:4 KEYSW, K4:5 KEYSW, K4:6 KEYSW, K4:7 KEYSW, K4:8 KEYSW, K4:9 KEYSW

Commit message: Rough out PCB layout
Parts:
- removed D0:8, D3:8, D4:8: D_Small_ALT, Diode_SMD:D_SOD-323_HandSoldering, symbol Device:D_Small_ALT
- removed K0:8, K3:8, K4:8: KEYSW, keyswitches_AO:Kailh_socket, symbol keyboard_parts:KEYSW
- K0:0, K0:1, K0:10, K0:11, K0:12, K0:13, K0:14, K0:15, K0:16, K0:2, K0:3, K0:4, K0:5, K0:6, K1:0, K1:1, K1:10, K1:11, K1:12, K1:13, K1:14, K1:15, K1:16, K1:2, K1:3, K1:4, K1:5, K1:6, K1:8, K2:0, K2:1, K2:10, K2:11, K2:12, K2:13, K2:14, K2:15, K2:16, K2:2, K2:3, K2:4, K2:5, K2:6, K2:8, K3:0, K3:1, K3:11, K3:12, K3:13, K3:14, K3:15, K3:16, K3:2, K3:3, K3:4, K3:5, K3:7, K3:9, K4:0, K4:1, K4:10, K4:11, K4:12, K4:13, K4:14, K4:15, K4:16, K4:2, K4:3, K4:4, K4:5, K4:6, K4:7, K4:9: footprint keyswitches_AO:Kailh_socket -> keyboard_parts_AO:Kailh_socket
Connections:
- wire segments 231 -> 222

Commit message: Start versioning here at v0.2
Parts:
- K0:0, K0:1, K0:10, K0:11, K0:12, K0:13, K0:14, K0:15, K0:16, K0:2, K0:3, K0:4, K0:5, K0:6, K1:0, K1:1, K1:10, K1:11, K1:12, K1:13, K1:14, K1:15, K1:16, K1:2, K1:3, K1:4, K1:5, K1:6, K1:8, K2:0, K2:1, K2:10, K2:11, K2:12, K2:13, K2:14, K2:15, K2:16, K2:2, K2:3, K2:4, K2:5, K2:6, K2:8, K3:0, K3:1, K3:11, K3:12, K3:13, K3:14, K3:15, K3:16, K3:2, K3:3, K3:4, K3:5, K3:7, K3:9, K4:0, K4:1, K4:10, K4:11, K4:12, K4:13, K4:14, K4:15, K4:16, K4:2, K4:3, K4:4, K4:5, K4:6, K4:7, K4:9: symbol keyboard_parts:KEYSW -> AODox-rescue:KEYSW-keyboard_parts

Commit message: Commit before pulling in from origin
Parts:
- D0:0, D0:1, D0:10, D0:11, D0:12, D0:13, D0:14, D0:15, D0:16, D0:2, D0:3, D0:4, D0:5, D0:6, D1:0, D1:1, D1:10, D1:11, D1:12, D1:13, D1:14, D1:15, D1:16, D1:2, D1:3, D1:4, D1:5, D1:6, D1:8, D2:0, D2:1, D2:10, D2:11, D2:12, D2:13, D2:14, D2:15, D2:16, D2:2, D2:3, D2:4, D2:5, D2:6, D2:8, D3:0, D3:1, D3:11, D3:12, D3:13, D3:14, D3:15, D3:16, D3:2, D3:3, D3:4, D3:5, D3:7, D3:9, D4:0, D4:1, D4:10, D4:11, D4:12, D4:13, D4:14, D4:15, D4:16, D4:2, D4:3, D4:4, D4:5, D4:6, D4:7, D4:9: symbol Device:D_Small_ALT -> AODox-rescue:D_Small_ALT-Device
